Commit message: update urdf and uf_ros_lib import

File: xarm_description/urdf/camera/realsense.gazebo.xacro (robot description, xacro)
@@ -1,6 +1,6 @@
 <?xml version="1.0"?>
 <robot xmlns:xacro="http://ros.org/wiki/xacro">
-  <xacro:macro name="realsense_gazebo" params="prefix:='' ">
-    <gazebo reference="${prefix}camera_depth_frame">
+  <xacro:macro name="realsense_gazebo" params="camera_prefix:='' ">
+    <gazebo reference="${camera_prefix}camera_depth_frame">
       <sensor name="cameradepth" type="depth">
         <camera name="camera">
@@ -25,5 +25,5 @@
       </sensor>
     </gazebo>
-    <gazebo reference="${prefix}camera_color_frame">
+    <gazebo reference="${camera_prefix}camera_color_frame">
       <sensor name="cameracolor" type="camera">
         <camera name="camera">
@@ -49,5 +49,5 @@
       </sensor>
     </gazebo>
-    <gazebo reference="${prefix}camera_left_ir_frame">
+    <gazebo reference="${camera_prefix}camera_left_ir_frame">
       <sensor name="cameraired1" type="camera">
         <camera name="camera">
@@ -73,5 +73,5 @@
       </sensor>
     </gazebo>
-    <gazebo reference="${prefix}camera_right_ir_frame">
+    <gazebo reference="${camera_prefix}camera_right_ir_frame">
       <sensor name="cameraired2" type="camera">
         <camera name="camera">

File: xarm_description/urdf/camera/realsense_d435i.urdf.xacro (robot description, xacro)
@@ -1,5 +1,5 @@
 <?xml version="1.0"?>
 <robot xmlns:xacro="http://ros.org/wiki/xacro">
-  <xacro:macro name="d435i_urdf" params="prefix:='' add_d435i_links:=false">
+  <xacro:macro name="d435i_urdf" params="prefix:='' camera_prefix:='' add_d435i_links:=false">
     <!-- define property -->
     <xacro:property name="M_PI" value="3.1415926535897931" />
@@ -16,56 +16,56 @@
     </link>
     <xacro:if value="${add_d435i_links}">
-      <link name="${prefix}camera_link"></link>
-      <link name="${prefix}camera_depth_frame"></link>
-      <link name="${prefix}camera_depth_optical_frame"></link>
-      <link name="${prefix}camera_color_frame"></link>
-      <link name="${prefix}camera_color_optical_frame"></link>
-      <link name="${prefix}camera_left_ir_frame"></link>
-      <link name="${prefix}camera_left_ir_optical_frame"></link>
-      <link name="${prefix}camera_right_ir_frame"></link>
-      <link name="${prefix}camera_right_ir_optical_frame"></link>
-      <joint name="${prefix}camera_link_joint" type="fixed">
+      <link name="${camera_prefix}camera_link"></link>
+      <link name="${camera_prefix}camera_depth_frame"></link>
+      <link name="${camera_prefix}camera_depth_optical_frame"></link>
+      <link name="${camera_prefix}camera_color_frame"></link>
+      <link name="${camera_prefix}camera_color_optical_frame"></link>
+      <link name="${camera_prefix}camera_left_ir_frame"></link>
+      <link name="${camera_prefix}camera_left_ir_optical_frame"></link>
+      <link name="${camera_prefix}camera_right_ir_frame"></link>
+      <link name="${camera_prefix}camera_right_ir_optical_frame"></link>
+      <joint name="${camera_prefix}camera_link_joint" type="fixed">
         <parent link="${prefix}link_eef" />
-        <child link="${prefix}camera_link" />
+        <child link="${camera_prefix}camera_link" />
         <origin xyz="0.06746 -0.0175 0.0237" rpy="${M_PI} ${-M_PI/2} 0" />
       </joint>
-      <joint name="${prefix}camera_depth_joint" type="fixed">
-        <parent link="${prefix}camera_link" />
-        <child link="${prefix}camera_depth_frame" />
+      <joint name="${camera_prefix}camera_depth_joint" type="fixed">
+        <parent link="${camera_prefix}camera_link" />
+        <child link="${camera_prefix}camera_depth_frame" />
         <origin xyz="0 0 0" rpy="0 0 0" />
       </joint>
-      <joint name="${prefix}camera_depth_optical_joint" type="fixed">
-        <parent link="${prefix}camera_depth_frame" />
-        <child link="${prefix}camera_depth_optical_frame" />
+      <joint name="${camera_prefix}camera_depth_optical_joint" type="fixed">
+        <parent link="${camera_prefix}camera_depth_frame" />
+        <child link="${camera_prefix}camera_depth_optical_frame" />
         <origin xyz="0 0 0" rpy="${-M_PI/2} 0 ${-M_PI/2}" />
       </joint>
-      <joint name="${prefix}camera_color_joint" type="fixed">
-        <parent link="${prefix}camera_link" />
-        <child link="${prefix}camera_color_frame" />
+      <joint name="${camera_prefix}camera_color_joint" type="fixed">
+        <parent link="${camera_prefix}camera_link" />
+        <child link="${camera_prefix}camera_color_frame" />
         <origin xyz="0 0.015 0" rpy="0 0 0" />
       </joint>
-      <joint name="${prefix}camera_color_optical_joint" type="fixed">
-        <parent link="${prefix}camera_color_frame" />
-        <child link="${prefix}camera_color_optical_frame" />
+      <joint name="${camera_prefix}camera_color_optical_joint" type="fixed">
+        <parent link="${camera_prefix}camera_color_frame" />
+        <child link="${camera_prefix}camera_color_optical_frame" />
         <origin xyz="0 0 0" rpy="${-M_PI/2} 0 ${-M_PI/2}" />
       </joint>
-      <joint name="${prefix}camera_left_ir_joint" type="fixed">
-        <parent link="${prefix}camera_link" />
-        <child link="${prefix}camera_left_ir_frame" />
+      <joint name="${camera_prefix}camera_left_ir_joint" type="fixed">
+        <parent link="${camera_prefix}camera_link" />
+        <child link="${camera_prefix}camera_left_ir_frame" />
         <origin xyz="0 0 0" rpy="0 0 0" />
       </joint>
-      <joint name="${prefix}camera_left_ir_optical_joint" type="fixed">
-        <parent link="${prefix}camera_left_ir_frame" />
-        <child link="${prefix}camera_left_ir_optical_frame" />
+      <joint name="${camera_prefix}camera_left_ir_optical_joint" type="fixed">
+        <parent link="${camera_prefix}camera_left_ir_frame" />
+        <child link="${camera_prefix}camera_left_ir_optical_frame" />
         <origin xyz="0 0 0" rpy="${-M_PI/2} 0 ${-M_PI/2}" />
       </joint>
-      <joint name="${prefix}camera_right_ir_joint" type="fixed">
-        <parent link="${prefix}camera_link" />
-        <child link="${prefix}camera_right_ir_frame" />
+      <joint name="${camera_prefix}camera_right_ir_joint" type="fixed">
+        <parent link="${camera_prefix}camera_link" />
+        <child link="${camera_prefix}camera_right_ir_frame" />
         <origin xyz="0 -0.050 0" rpy="0 0 0" />
       </joint>
-      <joint name="${prefix}camera_right_ir_optical_joint" type="fixed">
-        <parent link="${prefix}camera_right_ir_frame" />
-        <child link="${prefix}camera_right_ir_optical_frame" />
+      <joint name="${camera_prefix}camera_right_ir_optical_joint" type="fixed">
+        <parent link="${camera_prefix}camera_right_ir_frame" />
+        <child link="${camera_prefix}camera_right_ir_optical_frame" />
         <origin xyz="0 0 0" rpy="${-M_PI/2} 0 ${-M_PI/2}" />
       </joint>

File: xarm_description/urdf/xarm_device.urdf.xacro (robot description, xacro)
@@ -2,4 +2,5 @@
 <robot xmlns:xacro="http://ros.org/wiki/xacro" name="UF_ROBOT">
   <xacro:arg name="prefix" default=""/>
+  <xacro:arg name="camera_prefix" default="xarm_"/>
   <xacro:arg name="hw_ns" default="xarm"/>
   <xacro:arg name="limited" default="false"/>
@@ -41,5 +42,5 @@
   <!-- load xarm device -->
   <xacro:include filename="$(find xarm_description)/urdf/xarm_device_macro.xacro" />
-  <xacro:xarm_device prefix="$(arg prefix)" hw_ns="$(arg hw_ns)" limited="$(arg limited)"
+  <xacro:xarm_device prefix="$(arg prefix)" camera_prefix="$(arg camera_prefix)" hw_ns="$(arg hw_ns)" limited="$(arg limited)"
     effort_control="$(arg effort_control)" velocity_control="$(arg velocity_control)"
     add_gripper="$(arg add_gripper)" add_vacuum_gripper="$(arg add_vacuum_gripper)"

File: xarm_description/urdf/xarm_device_macro.xacro (robot description, xacro)
@@ -3,4 +3,5 @@
   <xacro:macro name="xarm_device" params="
     prefix:=''
+    camera_prefix:=''
     hw_ns:='xarm'
     limited:=false
@@ -204,8 +205,8 @@
       <!-- (xarm) Load RealSense D435i URDF -->
       <xacro:include filename="$(find xarm_description)/urdf/camera/realsense_d435i.urdf.xacro" />
-      <xacro:d435i_urdf prefix="${prefix}" add_d435i_links="${add_d435i_links}" />
+      <xacro:d435i_urdf prefix="${prefix}" camera_prefix="${camera_prefix}" add_d435i_links="${add_d435i_links}" />
       <xacro:if value="${add_d435i_links}">
         <xacro:include filename="$(find xarm_description)/urdf/camera/realsense.gazebo.xacro" />
-        <xacro:realsense_gazebo prefix="${prefix}" />
+        <xacro:realsense_gazebo camera_prefix="${camera_prefix}" />
       </xacro:if>
     </xacro:if>
@@ -214,5 +215,5 @@
     </xacro:unless>
     <joint name="${prefix}joint_eef" type="fixed">
-      <origin xyz="0 0 0" rpy="0 0 0" />
+      <origin xyz="0 0 0" rpy="0 0 0.785" />
       <parent link="${prefix}link${dof}" />
       <child link="${prefix}link_eef" />
