Commit message: add srdf path and rviz path parameters

File: xarm_description/urdf/xarm_device.urdf.xacro (robot description, xacro)
@@ -8,4 +8,5 @@
   <xacro:arg name="velocity_control" default="false"/>
   <xacro:arg name="add_gripper" default="false"/>
+  <xacro:arg name="add_robotiq" default="true"/>
   <xacro:arg name="add_vacuum_gripper" default="false"/>
   <xacro:arg name="add_bio_gripper" default="false"/>
@@ -44,5 +45,5 @@
   <xacro:xarm_device prefix="$(arg prefix)" camera_prefix="$(arg camera_prefix)" hw_ns="$(arg hw_ns)" limited="$(arg limited)"
     effort_control="$(arg effort_control)" velocity_control="$(arg velocity_control)"
-    add_gripper="$(arg add_gripper)" add_vacuum_gripper="$(arg add_vacuum_gripper)"
+    add_gripper="$(arg add_gripper)" add_robotiq="$(arg add_robotiq)" add_vacuum_gripper="$(arg add_vacuum_gripper)"
     add_bio_gripper="$(arg add_bio_gripper)" dof="$(arg dof)"
     ros2_control_plugin="$(arg ros2_control_plugin)" robot_type="$(arg robot_type)"

File: xarm_description/urdf/xarm_device_macro.xacro (robot description, xacro)
@@ -9,4 +9,5 @@
     velocity_control:=false
     add_gripper:=false
+    add_robotiq:=false
     add_vacuum_gripper:=false
     add_bio_gripper:=false
@@ -215,5 +216,5 @@
     </xacro:unless>
     <joint name="${prefix}joint_eef" type="fixed">
-      <origin xyz="0 0 0" rpy="0 0 0.785" />
+      <origin xyz="0 0 0" rpy="0 0 0.0" />
       <parent link="${prefix}link${dof}" />
       <child link="${prefix}link_eef" />
@@ -230,4 +231,18 @@
         <xacro:xarm_gripper_macro prefix="${prefix}" attach_to="${prefix}link_eef"
           ros2_control_plugin="${ros2_control_plugin}" dof="${dof}" hard_interface="${hard_interface}" />
+      </xacro:unless>
+    </xacro:if>
+    <xacro:if value="${add_robotiq}">
+      <xacro:if value="${robot_type == 'lite'}">
+        <!-- Load Lite Gripper Model URDF -->
+        <xacro:include filename="$(find xarm_description)/urdf/gripper/lite_gripper.urdf.xacro" />
+        <xacro:uflite_gripper_urdf prefix="${prefix}" attach_to="${prefix}link_eef" />
+      </xacro:if>
+      <xacro:unless value="${robot_type == 'lite'}">
+        <!-- Load XArm Gripper Model URDF -->
+        <xacro:include filename="$(find robotiq_description)/urdf/gripper/robotiq_2f_140_macro.urdf.xacro" />
+        <xacro:robotiq_gripper name="RobotiqGripperHardwareInterface" prefix="${prefix}" parent="${prefix}link_eef" use_fake_hardware="true">
+          <origin xyz="0 0 0" rpy="0 0 0" />
+        </xacro:robotiq_gripper>
       </xacro:unless>
     </xacro:if>
