Commit message: update octomap

File: xarm_description/urdf/gripper/xarm_gripper.urdf.xacro (robot description, xacro)
@@ -184,5 +184,5 @@
     <link name="${prefix}link_tcp" />
     <joint name="${prefix}joint_tcp" type="fixed">
-      <origin xyz="0 0 0.172" rpy="0 0 0" />
+      <origin xyz="0 0 0.165" rpy="0 0 0" />
       <parent link="${prefix}xarm_gripper_base_link" />
       <child link="${prefix}link_tcp" />

Commit message: change the position of link gripper

File: xarm_description/urdf/gripper/xarm_gripper.urdf.xacro (robot description, xacro)
@@ -184,5 +184,5 @@
     <link name="${prefix}link_tcp" />
     <joint name="${prefix}joint_tcp" type="fixed">
-      <origin xyz="0 0 0.165" rpy="0 0 0" />
+      <origin xyz="0 0 0.19" rpy="0 0 0" />
       <parent link="${prefix}xarm_gripper_base_link" />
       <child link="${prefix}link_tcp" />
