Commit message: add initial grasp pose in srdf

File: xarm_moveit_config/srdf/_xarm7_macro.srdf.xacro (robot description, xacro)
@@ -56,4 +56,13 @@
       <joint name="${prefix}joint5" value="0" />
       <joint name="${prefix}joint6" value="-1.5708" />
+      <joint name="${prefix}joint7" value="0" />
+    </group_state>
+    <group_state name="initial" group="${prefix}xarm7">
+      <joint name="${prefix}joint1" value="0" />
+      <joint name="${prefix}joint2" value="0" />
+      <joint name="${prefix}joint3" value="0" />
+      <joint name="${prefix}joint4" value="0" />
+      <joint name="${prefix}joint5" value="0" />
+      <joint name="${prefix}joint6" value="-0.785" />
       <joint name="${prefix}joint7" value="0" />
     </group_state>

Commit message: zhongguancun version

File: xarm_moveit_config/srdf/_xarm7_macro.srdf.xacro (robot description, xacro)
@@ -66,4 +66,13 @@
       <joint name="${prefix}joint6" value="-0.785" />
       <joint name="${prefix}joint7" value="0" />
+    </group_state>
+    <group_state name="base_moving" group="${prefix}xarm7">
+      <joint name="${prefix}joint1" value="-1.525" />
+      <joint name="${prefix}joint2" value="-1.026" />
+      <joint name="${prefix}joint3" value="-0.042" />
+      <joint name="${prefix}joint4" value="-0.044" />
+      <joint name="${prefix}joint5" value="0.215" />
+      <joint name="${prefix}joint6" value="-1.482" />
+      <joint name="${prefix}joint7" value="-0.143" />
     </group_state>
     <!-- gripper -->

Commit message: fix: table grasp pose; debug prints

File: xarm_moveit_config/srdf/_xarm7_macro.srdf.xacro (robot description, xacro)
@@ -75,4 +75,13 @@
       <joint name="${prefix}joint6" value="-1.482" />
       <joint name="${prefix}joint7" value="-0.143" />
+    </group_state>
+    <group_state name="table_grasp" group="${prefix}xarm7">
+      <joint name="${prefix}joint1" value="0." />
+      <joint name="${prefix}joint2" value="-0.4187" />
+      <joint name="${prefix}joint3" value="0." />
+      <joint name="${prefix}joint4" value="1.709" />
+      <joint name="${prefix}joint5" value="0." />
+      <joint name="${prefix}joint6" value="1.343" />
+      <joint name="${prefix}joint7" value="0." />
     </group_state>
     <!-- gripper -->
